Commit message: urdf

File: PSA-ros/aulas/controlo/pend.urdf (robot description, URDF)
Before this commit: robot pend_robot, 5 links, 4 joints
Links:
- link ball_link: mass None -> 10
- link base_link: mass None -> 100

Commit message: control.yaml

File: PSA-ros/aulas/controlo/pend.urdf (robot description, URDF)
Before this commit: robot pend_robot, 6 links, 5 joints
Joints:
- joint motor_joint: type revolute -> continuous

Commit message: control.yaml

File: PSA-ros/aulas/controlo/pend.urdf (robot description, URDF)
Before this commit: robot pend_robot, 6 links, 5 joints
Joints:
- joint motor_joint: type continuous -> revolute

Commit message: control.yaml

File: PSA-ros/aulas/controlo/pend.urdf (robot description, URDF)
Before this commit: robot pend_robot, 6 links, 5 joints
Links:
- link body_link: mass None -> 100
